Commit message: frame issue

File: urdf/jackal.urdf.xacro (robot description, xacro)
@@ -3,5 +3,5 @@
      into Gazebo using robot state publisher.
      Requires the arguments: $namespace, $id -->
-<robot name="jackal" xmlns:xacro="http://www.ros.org/wiki/xacro">
+<robot name="$(arg namespace)" xmlns:xacro="http://www.ros.org/wiki/xacro">
   <xacro:property name="PI"                        value="3.1415926535897931" />
   <xacro:property name="wheelbase"                 value="0.262" />
@@ -79,4 +79,10 @@
     <origin xyz="${-wheelbase/2} ${-track/2} ${wheel_vertical_offset}" rpy="0 0 0" />
   </xacro:wheel>
+  <!-- <link name="odom_link"></link>
+  <joint name="odom_joint" type="fixed">
+    <origin xyz="0 0 0" rpy="0 0 0" />
+    <parent link="odom"/>
+    <child link="base_link" />
+  </joint> -->
   <link name="base_link"></link>
   <joint name="base_link_joint" type="fixed">

Commit message: multiple jackal

File: urdf/jackal.urdf.xacro (robot description, xacro)
@@ -79,10 +79,4 @@
     <origin xyz="${-wheelbase/2} ${-track/2} ${wheel_vertical_offset}" rpy="0 0 0" />
   </xacro:wheel>
-  <!-- <link name="odom_link"></link>
-  <joint name="odom_joint" type="fixed">
-    <origin xyz="0 0 0" rpy="0 0 0" />
-    <parent link="odom"/>
-    <child link="base_link" />
-  </joint> -->
   <link name="base_link"></link>
   <joint name="base_link_joint" type="fixed">
