Commit message: jackal+vlp16 + gazebo_maps

File: bigbot_description/urdf/jackal_all.urdf.xacro (robot description, xacro)
@@ -223,5 +223,5 @@
   </joint>
   <!-- Adding the ULU02 -->
-  <link name="enclosure_mount_link">
+  <!-- <link name="enclosure_mount_link">
     <visual>
       <origin xyz="0 0 0" rpy="0 0 0"/>
@@ -250,5 +250,5 @@
     <child link="zed_camera_center" />
     <origin xyz="0.175 0 0.115" />
-  </joint>
+  </joint> -->
   <!-- Adding lidar frame -->
   <!-- <link name="lidar_mounting_frame">
@@ -313,3 +313,8 @@
   <!-- Optional custom includes. -->
   <xacro:include filename="$(optenv JACKAL_URDF_EXTRAS empty.urdf)" />
+  <!-- VLP-16 -->
+  <xacro:include filename="$(find velodyne_description)/urdf/VLP-16.urdf.xacro"/>
+  <VLP-16 parent="base_link" name="velodyne" topic="/velodyne_points" hz="10" samples="360" gpu="true" lasers="16" max_range="100">
+    <origin xyz="0 0 0.4" rpy="0 0 0" />
+  </VLP-16>
 </robot>
